Commit message: removing instances of map1

File: excuse_me_pkg/urdf/excuse_me.urdf (robot description, URDF)
Before this commit: robot origins, 26 links, 25 joints
Links:
- removed link map1
- added link map; visual box size=0 0 0
Joints:
- joint base_link_to_mapVeh: parent map1 -> map

Commit message: frame change: map is now map_veh and hd_map is now map. This allows me to leave all the autoware stuff alone and just make changes to the gps/csv generator/custome tracker code.

File: excuse_me_pkg/urdf/excuse_me.urdf (robot description, URDF)
Before this commit: robot origins, 26 links, 25 joints
Links:
- removed link map
- added link map_veh; visual box size=0 0 0
Joints:
- removed joint base_link_to_mapVeh
- added joint base_link_to_map_veh: type fixed, parent map_veh, child base_link, origin xyz=0 0 0 rpy=0 0 0

Commit message: debugging stuff, extra launch file to use only top lidar, extra frame added to gpsins

File: excuse_me_pkg/urdf/excuse_me.urdf (robot description, URDF)
Before this commit: robot origins, 26 links, 25 joints
Links:
- removed link map_veh

Commit message: adds package to visualize the subject vehicle velocity in rviz using the current velocity and current pose topics publishd by gpsins_localizer

File: excuse_me_pkg/urdf/excuse_me.urdf (robot description, URDF)
Before this commit: robot origins, 25 links, 25 joints
Links:
- added link map_veh; visual box size=0 0 0
